Commit message: feat: param lidar and kinect

File: nebula-ws/src/axebot_description/urdf/lidar.xacro (robot description, xacro)
@@ -4,5 +4,5 @@
         <parent link="base_link"/>
         <child link="laser_frame"/>
-        <origin xyz="0.122 0 0.212" rpy="0 0 0"/>
+        <origin xyz="-0.13 0 0.31" rpy="0 0 0"/>
     </joint>
     <link name="laser_frame">
@@ -10,11 +10,4 @@
             <geometry>
                 <cylinder radius="0.05" length="0.04"/>
-            </geometry>
-            <material name="black"/>
-        </visual>
-        <visual>
-            <origin xyz="0 0 -0.05"/>
-            <geometry>
-                <cylinder radius="0.01" length="0.1"/>
             </geometry>
             <material name="black"/>
