Commit message: feat: add launch file gazebo

File: nebula-ws/src/axebot_description/urdf/axebot.urdf.xacro (robot description, xacro)
@@ -17,8 +17,8 @@
     <xacro:property name="wheel_thickness" value="0.01905" />
     <xacro:property name="motor_shaft_length" value="0.005475"/>
-    <xacro:include filename="$(find nebula_description)/urdf/wheel.urdf.xacro"/>
-    <xacro:include filename="$(find nebula_description)/urdf/materials.urdf.xacro"/>
-    <xacro:include filename="$(find nebula_description)/urdf/gazebo.urdf.xacro"/>
-    <xacro:include filename="$(find nebula_description)/urdf/ros2_control.urdf.xacro"/>
+    <xacro:include filename="$(find axebot_description)/urdf/wheel.urdf.xacro"/>
+    <xacro:include filename="$(find axebot_description)/urdf/materials.urdf.xacro"/>
+    <!-- <xacro:include filename="$(find axebot_description)/urdf/gazebo.urdf.xacro"/>
+    <xacro:include filename="$(find axebot_description)/urdf/ros2_control.urdf.xacro"/> -->
     <link name="base_link"></link>
     <joint name="base_link_joint" type="fixed">

File: nebula-ws/src/axebot_description/urdf/wheel.urdf.xacro (robot description, xacro)
@@ -27,5 +27,5 @@
                 <origin xyz="0.0 0.0 0.0" rpy="0.0 0.0 0.0"/>
                 <geometry>
-                    <mesh filename="file://$(find nebula_description)/meshes/roller.stl"/>
+                    <mesh filename="file://$(find axebot_description)/meshes/roller.stl"/>
                 </geometry>
                 <material name="green"/>
@@ -34,5 +34,5 @@
                 <origin xyz="0.0 0.0 0.0" rpy="0.0 0.0 0.0"/>
                 <geometry>
-                    <mesh filename="file://$(find nebula_description)/meshes/roller.stl"/>
+                    <mesh filename="file://$(find axebot_description)/meshes/roller.stl"/>
                 </geometry>
             </collision>
@@ -90,5 +90,5 @@
                 <origin xyz="0.0 0.0 0.0" rpy="0.0 0.0 0.0"/>
                 <geometry>
-                    <mesh filename="file://$(find nebula_description)/meshes/rim.stl"/>
+                    <mesh filename="file://$(find axebot_description)/meshes/rim.stl"/>
                 </geometry>
                 <material name="grey"/>
@@ -97,5 +97,5 @@
                 <origin xyz="0.0 0.0 0.0" rpy="0.0 0.0 0.0"/>
                 <geometry>
-                    <mesh filename="file://$(find nebula_description)/meshes/wheel-collision.dae"/>
+                    <mesh filename="file://$(find axebot_description)/meshes/wheel-collision.dae"/>
                 </geometry>
             </collision>

Commit message: feat: ros2 control works gazebo

File: nebula-ws/src/axebot_description/urdf/axebot.urdf.xacro (robot description, xacro)
@@ -19,6 +19,6 @@
     <xacro:include filename="$(find axebot_description)/urdf/wheel.urdf.xacro"/>
     <xacro:include filename="$(find axebot_description)/urdf/materials.urdf.xacro"/>
-    <!-- <xacro:include filename="$(find axebot_description)/urdf/gazebo.urdf.xacro"/>
-    <xacro:include filename="$(find axebot_description)/urdf/ros2_control.urdf.xacro"/> -->
+    <xacro:include filename="$(find axebot_description)/urdf/gazebo.urdf.xacro"/>
+    <xacro:include filename="$(find axebot_description)/urdf/ros2_control.urdf.xacro"/>
     <link name="base_link"></link>
     <joint name="base_link_joint" type="fixed">

File: nebula-ws/src/axebot_description/urdf/gazebo.urdf.xacro (robot description, xacro)
@@ -1,21 +1,21 @@
 <robot xmlns:xacro="http://www.ros.org/wiki/xacro" name="axebot">
-    <transmission name="wheel_1_transmission">
+    <transmission name="wheel1_transmission">
         <plugin>transmission_interface/SimpleTransmission</plugin>
-        <actuator name="wheel_1_motor" role="actuator_1"/>
-        <joint name="wheel_1_joint" role="joint_1"/>
+        <actuator name="wheel1_motor" role="actuator1"/>
+        <joint name="wheel1_joint" role="joint1">
             <mechanicalReduction>1.0</mechanicalReduction>
         </joint>
     </transmission>
-    <transmission name="wheel_2_transmission">
+    <transmission name="wheel2_transmission">
         <plugin>transmission_interface/SimpleTransmission</plugin>
-        <actuator name="wheel_2_motor" role="actuator_2"/>
-        <joint name="wheel_2_joint" role="joint_2"/>
+        <actuator name="wheel2_motor" role="actuator2"/>
+        <joint name="wheel2_joint" role="joint2">
             <mechanicalReduction>1.0</mechanicalReduction>
         </joint>
     </transmission>
-    <transmission name="wheel_3_transmission">
+    <transmission name="wheel3_transmission">
         <plugin>transmission_interface/SimpleTransmission</plugin>
-        <actuator name="wheel_3_motor" role="actuator_3"/>
-        <joint name="wheel_3_joint" role="joint_3"/>
+        <actuator name="wheel3_motor" role="actuator3"/>
+        <joint name="wheel3_joint" role="joint3">
             <mechanicalReduction>1.0</mechanicalReduction>
         </joint>
@@ -26,5 +26,5 @@
     <gazebo reference="wheel1_link">
         <material>Gazebo/Grey</material>
-        <fdir1>0 1 0"</fdir1>
+        <fdir1>0 1 0</fdir1>
         <mu1>1.7</mu1>
         <mu2>0.2</mu2>
@@ -32,5 +32,5 @@
     <gazebo reference="wheel2_link">
         <material>Gazebo/Grey</material>
-        <fdir1>0 1 0"</fdir1>
+        <fdir1>0 1 0</fdir1>
         <mu1>1.7</mu1>
         <mu2>0.2</mu2>
@@ -38,25 +38,14 @@
     <gazebo reference="wheel3_link">
         <material>Gazebo/Grey</material>
-        <fdir1>0 1 0"</fdir1>
+        <fdir1>0 1 0</fdir1>
         <mu1>1.7</mu1>
         <mu2>0.2</mu2>
     </gazebo>
-</robot>
-    <!--
     <gazebo>
         <plugin filename="libgazebo_ros2_control.so" name="gazebo_ros2_control">
             <robot_param>robot_description</robot_param>
             <robot_param_node>robot_state_publisher</robot_param_node>
-            <!--  <parameters>$(find axebot_control)/config/omnidirectional_controller.yaml</parameters> -->
-        </plugin>
-        <plugin filename="libgazebo_ros_p3d.so" name="gazebo_ros_p3d" >
-            <ros>
-                <namespace>gazebo_ground_truth</namespace>
-            </ros>
-            <frame_name>world</frame_name>
-            <body_name>base_link</body_name>
-            <update_rate>50.0</update_rate>
-            <gaussian_noise>0.01</gaussian_noise>
+            <parameters>$(find nebula_controller)/config/nebula_controllers.yaml</parameters>
         </plugin>
     </gazebo>
-    -->
+</robot>

Commit message: feat: done mapping room

File: nebula-ws/src/axebot_description/urdf/axebot.urdf.xacro (robot description, xacro)
@@ -22,5 +22,13 @@
     <xacro:include filename="$(find axebot_description)/urdf/gazebo.urdf.xacro"/>
     <xacro:include filename="$(find axebot_description)/urdf/ros2_control.urdf.xacro"/>
+    <xacro:include filename="$(find axebot_description)/urdf/lidar.xacro"/>
     <link name="base_link"></link>
+    <!-- Base Footptint -->
+    <link name="base_footprint"></link>
+    <joint name="base_footprint_joint" type="fixed">
+        <origin xyz="0 0 0" rpy="0 0 0" />
+        <parent link="base_link"/>
+        <child link="base_footprint" />
+    </joint>
     <joint name="base_link_joint" type="fixed">
         <origin xyz="0 0 ${robot_height}" rpy="0 0 0" />

Commit message: feat: add scan 2d from 3d kinect

File: nebula-ws/src/axebot_description/urdf/axebot.urdf.xacro (robot description, xacro)
@@ -22,5 +22,6 @@
     <xacro:include filename="$(find axebot_description)/urdf/gazebo.urdf.xacro"/>
     <xacro:include filename="$(find axebot_description)/urdf/ros2_control.urdf.xacro"/>
-    <xacro:include filename="$(find axebot_description)/urdf/lidar.xacro"/>
+    <!-- <xacro:include filename="$(find axebot_description)/urdf/lidar.xacro"/> -->
+    <xacro:include filename="$(find axebot_description)/urdf/depth_camera.xacro"/>
     <link name="base_link"></link>
     <!-- Base Footptint -->

File: nebula-ws/src/axebot_description/urdf/depth_camera.xacro (robot description, xacro)
@@ -12,5 +12,5 @@
         <parent link="base_link"/>
         <child link="camera_link"/>
-        <origin xyz="0.0 0 0.08" rpy="0 0 0"/>
+        <origin xyz="0.0 0 0.5" rpy="0 0 0"/>
     </joint>
     <joint name="camera_optical_joint" type="fixed">

Commit message: feat: add kinect link and fix param robot

File: nebula-ws/src/axebot_description/urdf/axebot.urdf.xacro (robot description, xacro)
@@ -7,7 +7,7 @@
     <xacro:property name="chassis_mass" value="1.074"/>
     <xacro:property name="chassis_height" value="0.04"/>
-    <xacro:property name="robot_height" value="0.053"/>
-    <xacro:property name="wheel_mass" value="0.105" />
-    <xacro:property name="wheel_radius" value="0.0508" />
+    <xacro:property name="robot_height" value="0.075"/>
+    <xacro:property name="wheel_mass" value="1.105" />
+    <xacro:property name="wheel_radius" value="0.15" />
     <xacro:property name="motor_shaft_radius" value="0.002" />
     <xacro:property name="shaft_mass" value="0.001" />
@@ -15,5 +15,5 @@
     motor shaft length must be equal to the robot radius L = 0.1 m used in the
     kinematic model -->
-    <xacro:property name="chassis_radius" value="0.085"/>
+    <xacro:property name="chassis_radius" value="0.28867"/>
     <xacro:property name="wheel_thickness" value="0.01905" />
     <xacro:property name="motor_shaft_length" value="0.005475"/>

File: nebula-ws/src/axebot_description/urdf/depth_camera.xacro (robot description, xacro)
@@ -4,5 +4,5 @@
         <visual>
             <geometry>
-                <box size="0.010 0.03 0.03"/>
+                <box size="0.066 0.249 0.067"/>
             </geometry>
             <material name="red"/>
@@ -12,5 +12,5 @@
         <parent link="base_link"/>
         <child link="camera_link"/>
-        <origin xyz="0.0 0 0.5" rpy="0 0 0"/>
+        <origin xyz="-0.13 0 0.25" rpy="0 0 0"/>
     </joint>
     <joint name="camera_optical_joint" type="fixed">
@@ -34,6 +34,6 @@
                 </image>
                 <clip>
-                    <near>0.05</near>
-                    <far>8.0</far>
+                    <near>0.04</near>
+                    <far>5.0</far>
                 </clip>
             </camera>

File: nebula-ws/src/axebot_description/urdf/wheel.urdf.xacro (robot description, xacro)
@@ -1,5 +1,5 @@
 <?xml version="1.0"?>
 <robot xmlns:xacro="http://www.ros.org/wiki/xacro">
-    <xacro:property name="distance_to_roller_center" value="0.04645"/>
+    <xacro:property name="distance_to_roller_center" value="0.07"/>
     <xacro:macro name="inertial_cylinder" params="mass length radius *origin">
         <inertial>

Commit message: error: odom

File: nebula-ws/src/axebot_description/urdf/axebot.urdf.xacro (robot description, xacro)
@@ -3,11 +3,11 @@
     <xacro:arg name="is_sim" default="true"/>
     <xacro:arg name="only_one_wheel" default="false"/>
-    <!-- Constants for wheel mechanical parameters -->
+   <!-- Constants for wheel mechanical parameters -->
     <xacro:property name="PI" value="3.1415926535897931"/>
     <xacro:property name="chassis_mass" value="1.074"/>
     <xacro:property name="chassis_height" value="0.04"/>
-    <xacro:property name="robot_height" value="0.075"/>
-    <xacro:property name="wheel_mass" value="1.105" />
-    <xacro:property name="wheel_radius" value="0.15" />
+    <xacro:property name="robot_height" value="0.053"/>
+    <xacro:property name="wheel_mass" value="0.105" />
+    <xacro:property name="wheel_radius" value="0.0508" />
     <xacro:property name="motor_shaft_radius" value="0.002" />
     <xacro:property name="shaft_mass" value="0.001" />
@@ -15,5 +15,5 @@
     motor shaft length must be equal to the robot radius L = 0.1 m used in the
     kinematic model -->
-    <xacro:property name="chassis_radius" value="0.28867"/>
+    <xacro:property name="chassis_radius" value="0.085"/>
     <xacro:property name="wheel_thickness" value="0.01905" />
     <xacro:property name="motor_shaft_length" value="0.005475"/>

File: nebula-ws/src/axebot_description/urdf/wheel.urdf.xacro (robot description, xacro)
@@ -1,5 +1,5 @@
 <?xml version="1.0"?>
 <robot xmlns:xacro="http://www.ros.org/wiki/xacro">
-    <xacro:property name="distance_to_roller_center" value="0.07"/>
+    <xacro:property name="distance_to_roller_center" value="0.04645"/>
     <xacro:macro name="inertial_cylinder" params="mass length radius *origin">
         <inertial>

Commit message: feat: nav2 with updated robot size

File: nebula-ws/src/axebot_description/urdf/axebot.urdf.xacro (robot description, xacro)
@@ -9,5 +9,5 @@
     <xacro:property name="robot_height" value="0.053"/>
     <xacro:property name="wheel_mass" value="0.105" />
-    <xacro:property name="wheel_radius" value="0.0508" />
+    <xacro:property name="wheel_radius" value="0.072687795" />
     <xacro:property name="motor_shaft_radius" value="0.002" />
     <xacro:property name="shaft_mass" value="0.001" />
@@ -15,5 +15,5 @@
     motor shaft length must be equal to the robot radius L = 0.1 m used in the
     kinematic model -->
-    <xacro:property name="chassis_radius" value="0.085"/>
+    <xacro:property name="chassis_radius" value="0.264145"/>
     <xacro:property name="wheel_thickness" value="0.01905" />
     <xacro:property name="motor_shaft_length" value="0.005475"/>

File: nebula-ws/src/axebot_description/urdf/wheel.urdf.xacro (robot description, xacro)
@@ -1,5 +1,5 @@
 <?xml version="1.0"?>
 <robot xmlns:xacro="http://www.ros.org/wiki/xacro">
-    <xacro:property name="distance_to_roller_center" value="0.04645"/>
+    <xacro:property name="distance_to_roller_center" value="0.068337795"/>
     <xacro:macro name="inertial_cylinder" params="mass length radius *origin">
         <inertial>
