Commit message: feat: using depthimage only, without pointcloud

File: nebula-ws/src/axebot_description/urdf/depth_camera.xacro (robot description, xacro)
@@ -20,4 +20,10 @@
     </joint>
     <link name="camera_link_optical"></link>
+    <link name="camera_depth_frame"/>
+    <joint name="camera_laser_joint" type="fixed">
+        <parent link="camera_link"/>
+        <child link="camera_depth_frame"/>
+        <origin xyz="0 0 0" rpy="0 0 0"/>
+    </joint>
     <gazebo reference="camera_link">
         <material>Gazebo/Red</material>
